File: OrangePiZero2_expboard/opi-hat.kicad_pcb (KiCad board)
At the start: 2 copper layers, 56.9 x 63.9 mm, 40 parts, among them J1 Hydreon, J2 I2C, J3 SPI, J4 12Vin, J5 USB_C_Receptacle_USB2.0, J6 USB_B, J7 5Vout, U1 PC817, U2 LM2576-5.0, U3 LM1117-3.3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

Commit message: fixed boards on new kicad
Parts:
- added D2: CESD3V3, Diode_SMD:D_SOD-323_HandSoldering, B.Cu at (93.0, 94.4)
- added TP10: LoL, TestPoint:TestPoint_THTPad_1.0x1.0mm_Drill0.5mm, F.Cu at (104.5, 53.0)
- added TP11: LoR, TestPoint:TestPoint_THTPad_1.0x1.0mm_Drill0.5mm, F.Cu at (106.6, 53.0)
- added TP12: Lgnd, TestPoint:TestPoint_THTPad_1.0x1.0mm_Drill0.5mm, F.Cu at (104.5, 55.0)
- added TP13: GND, TestPoint:TestPoint_THTPad_2.5x2.5mm_Drill1.2mm, F.Cu at (128.3, 88.8)
- added TP14: GND, TestPoint:TestPoint_THTPad_2.5x2.5mm_Drill1.2mm, F.Cu at (94.6, 56.5)
- added TP15: GND, TestPoint:TestPoint_THTPad_2.5x2.5mm_Drill1.2mm, F.Cu at (98.2, 56.5)
- added TP16: 3V3, TestPoint:TestPoint_THTPad_2.5x2.5mm_Drill1.2mm, F.Cu at (124.5, 88.8)
- added TP17: GND, TestPoint:TestPoint_THTPad_2.5x2.5mm_Drill1.2mm, F.Cu at (101.7, 56.5)
- added TP5: PC10, TestPoint:TestPoint_THTPad_2.5x2.5mm_Drill1.2mm, F.Cu at (128.9, 104.5)
- added TP6: PC1, TestPoint:TestPoint_THTPad_2.5x2.5mm_Drill1.2mm, F.Cu at (101.7, 53.0)
- added TP8: PI6, TestPoint:TestPoint_THTPad_2.5x2.5mm_Drill1.2mm, F.Cu at (94.6, 53.0)
- added TP9: PI16, TestPoint:TestPoint_THTPad_2.5x2.5mm_Drill1.2mm, F.Cu at (98.2, 53.0)
- moved TP2 0.85 mm to (128.3, 92.3)
- moved TP4 0.38 mm to (124.5, 92.3)
Connections:
- X1 pad 26: unconnected-(X1-Pad26) -> Net-(TP5-Pad1)
- X1 pad 33: unconnected-(X1-Pad33) -> Net-(TP11-Pad1)
- X1 pad 34: unconnected-(X1-Pad34) -> Net-(TP10-Pad1)
- X1 pad 36: unconnected-(X1-Pad36) -> Net-(TP6-Pad1)
- X1 pad 37: unconnected-(X1-Pad37) -> Net-(TP9-Pad1)
- X1 pad 38: unconnected-(X1-Pad38) -> Net-(TP8-Pad1)
Routing:
- net GND: track 366.6 -> 373.4 mm
- net Net-(TP11-Pad1): track 0.00 -> 5.02 mm
- net Net-(TP10-Pad1): track 0.00 -> 4.64 mm
- net Net-(TP8-Pad1): track 0.00 -> 4.54 mm
- net Net-(TP9-Pad1): track 0.00 -> 4.12 mm
- net Net-(TP6-Pad1): track 0.00 -> 3.70 mm
- net Net-(TP5-Pad1): track 0.00 -> 3.52 mm
- net +3.3V: track 72.2 -> 75.6 mm
- net /SCK: track 20.2 -> 21.7 mm
- net /SDA: track 16.1 -> 15.3 mm
Other:
- board text added: "1"
- board text added: "12V Tx GND"
- board text added: "2"
- board text added: "25"
- board text added: "26"
- board text added: "27"
- board text added: "39"
- board text added: "3V3 CLK MISO MOSI GND"
- board text added: "GND"
- board text added: "GND SDA SCK 3V3"
