File: OrangePiZero_expboard/opi-hat.kicad_sch (KiCad schematic)
At the start: 36 parts, among them J1 Hydreon, J2 I2C, J3 SPI, J4 12Vin, J5 USB_C_Receptacle_USB2.0, J6 USB_B, J7 5Vout, U1 PC817, U2 LM2576-5.0, U3 LM1117-3.3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

Commit message: fixed boards on new kicad
Parts:
- added D2: CESD3V3, Diode_SMD:D_SOD-323_HandSoldering, symbol Diode:ESD9B3.3ST5G
Connections:
- net GND: now also D2.2 (A2)
- net SCK: now also D2.1 (A1)
